File: src/kicad files/radio.kicad_pcb (KiCad board)
At the start: 2 copper layers, 97.6 x 67.8 mm, 37 parts, among them CN1 PJ-3200, J1 Conn_01x04_Pin, J2 Conn_01x06_Pin, J4 Speaker 1, J5 Speaker 2, SW3 SW_Push, SW4 SW_Push, SW5 SW_Push, SW6 SW_Push, U1 XIAO-RP2040-DIP, U2 RDA5807MRRD-102V2.0, U3 TDA2822NBD, U4 TSOP38238, U5 SX1278, Y2 Crystal

Commit message: updated with changes
Parts:
- J1: value Conn_01x04_Pin -> 0.96in OLED Display
- J2: value Conn_01x06_Pin -> MicroSD Card Module
- moved RV1 32.7 mm to (129.1, 96.8), turned to 90 degrees
- moved RV2 18.2 mm to (117.6, 96.8), turned to 90 degrees
- moved CN1 15.0 mm to (109.4, 92.4), turned to 90 degrees
- moved H3 1.34 mm to (85.4, 95.2)
Routing:
- net Net-(U3-IN2): track 64.3 -> 90.5 mm, vias 2 -> 3
- net Net-(U3-IN1): track 86.9 -> 111.3 mm, vias 9 -> 8
- net /ANT: track 110.5 -> 133.1 mm, vias 7 -> 11
- net /LOUT: track 29.5 -> 38.6 mm, vias 5 -> 6
- net /ROUT: track 29.2 -> 20.4 mm
- net GND: track 271.9 -> 267.0 mm, vias 7 -> 11
- net Net-(U2-ANT): track 19.1 -> 16.1 mm, vias 0 -> 1
